Commit message: Add navigation package

File: simple4wd_description/urdf/accessories/hokuyo_laser.urdf.xacro (robot description, xacro)
@@ -2,6 +2,5 @@
 <robot name="simple4wd"
   xmlns:xacro="http://www.ros.org/wiki/xacro">
-  <xacro:macro name="hokuyo_laser" params="prefix parent_link trans_x trans_y trans_z
-   robot_namespace:=/simple4wd frame:=laser topic:=scan">
+  <xacro:macro name="hokuyo_laser" params="prefix parent_link trans_x trans_y trans_z">
     <link name="${prefix}_hokuyo_link">
       <collision>
@@ -63,6 +62,6 @@
         </ray>
         <plugin name="gazebo_ros_laser" filename="libgazebo_ros_laser.so">
-          <topicName>${topic}</topicName>
-          <frameName>${frame}</frameName>
+          <topicName>/simple4wd/laser/scan</topicName>
+          <frameName>${prefix}_hokuyo_link</frameName>
           <robotNamespace>${robot_namespace}</robotNamespace>
         </plugin>

File: simple4wd_description/urdf/simple4wd.urdf.xacro (robot description, xacro)
@@ -5,8 +5,18 @@
   <xacro:include filename="$(find simple4wd_description)/urdf/wheel.urdf.xacro" />
   <xacro:include filename="$(find simple4wd_description)/urdf/accessories/hokuyo_laser.urdf.xacro" />
-  <!-- ROS Control Plugin -->
+  <!-- Gazebo Plugins -->
   <gazebo>
     <plugin name="gazebo_ros_control" filename="libgazebo_ros_control.so">
       <robotNamespace>/simple4wd</robotNamespace>
+    </plugin>
+  </gazebo>
+  <gazebo>
+    <plugin name="imu_plugin" filename="libgazebo_ros_imu.so">
+      <alwaysOn>true</alwaysOn>
+      <bodyName>chassis_link</bodyName>
+      <topicName>imu</topicName>
+      <serviceName>imu_service</serviceName>
+      <gaussianNoise>0.0</gaussianNoise>
+      <updateRate>20.0</updateRate>
     </plugin>
   </gazebo>
