Commit message: Played around with rtabmap

File: simple4wd_description/urdf/accessories/kinect_camera.urdf.xacro (robot description, xacro)
@@ -37,4 +37,12 @@
       <child link="${prefix}_camera_link"/>
     </joint>
+    <!-- Fixes bug with depth camera frame
+      https://answers.ros.org/question/218395/libgazebo_ros_openni_kinectso-depth-pointcloud-wrong-tf/ -->
+    <link name="${prefix}_camera_depth_link"/>
+    <joint name="${prefix}_camera_depth_joint" type="fixed">
+      <origin xyz="0 0 0" rpy="${-PI/2} 0 ${-PI/2}"/>
+      <parent link="${prefix}_camera_link"/>
+      <child link="${prefix}_camera_depth_link"/>
+    </joint>
     <gazebo reference="${prefix}_camera_link">
       <sensor name="${prefix}_camera" type="depth">
@@ -62,5 +70,5 @@
           <depthImageInfoTopicName>/simple4wd/${prefix}_camera/depth/camera_info</depthImageInfoTopicName>
           <pointCloudTopicName>/simple4wd/${prefix}_camera/depth/points</pointCloudTopicName>
-          <frameName>${prefix}_camera_link</frameName>
+          <frameName>${prefix}_camera_depth_link</frameName>
           <pointCloudCutoff>0.5</pointCloudCutoff>
           <pointCloudCutoffMax>3.0</pointCloudCutoffMax>

File: simple4wd_description/urdf/simple4wd.urdf.xacro (robot description, xacro)
@@ -99,5 +99,5 @@
   />
   <xacro:kinect_camera prefix="kinect" parent_link="chassis_link">
-    <origin xyz="${BASE_LENGTH/2} 0 ${BASE_HEIGHT}" rpq="${PI} 0 0" />
+    <origin xyz="${BASE_LENGTH/2} 0 ${BASE_HEIGHT + 0.1}" rpq="${PI} ${-PI/4} 0" />
   </xacro:kinect_camera>
 </robot>
