Commit message: Add laser sensor

File: simple4wd_description/urdf/simple4wd.urdf.xacro (robot description, xacro)
@@ -2,6 +2,8 @@
 <robot name="simple4wd"
   xmlns:xacro="http://www.ros.org/wiki/xacro">
-  <!-- Import wheel element -->
+  <!-- Import urdf.xacro files -->
   <xacro:include filename="$(find simple4wd_description)/urdf/wheel.urdf.xacro" />
+  <xacro:include filename="$(find simple4wd_description)/urdf/accessories/hokuyo_laser.urdf.xacro" />
+  <!-- ROS Control Plugin -->
   <gazebo>
     <plugin name="gazebo_ros_control" filename="libgazebo_ros_control.so">
@@ -22,6 +24,13 @@
     <color rgba="0 1.0 1.0 1.0"/>
   </material>
+  <!-- Dummy link that doesn't have inertia -->
+  <link name="base_link" />
+  <joint name="base_link_joint" type="fixed">
+    <parent link="base_link"/>
+    <child link="chassis_link" />
+    <origin xyz="0 0 0" rpy="0 0 0" />
+  </joint>
   <!-- Robot Base (front is facing positive x) -->
-  <link name="base_link">
+  <link name="chassis_link">
     <visual>
       <geometry>
@@ -46,5 +55,5 @@
   <!-- Wheels -->
   <xacro:wheel
-    name_link="left_front_wheel" parent_link="base_link"
+    name_link="left_front_wheel" parent_link="chassis_link"
     mass="${WHEEL_MASS}" radius="${WHEEL_RADIUS}" width="${WHEEL_WIDTH}"
     translate_x="${BASE_WIDTH/2 - 2*WHEEL_RADIUS}"
@@ -53,5 +62,5 @@
   />
   <xacro:wheel
-    name_link="right_back_wheel" parent_link="base_link"
+    name_link="right_back_wheel" parent_link="chassis_link"
     mass="${WHEEL_MASS}" radius="${WHEEL_RADIUS}" width="${WHEEL_WIDTH}"
     translate_x="${-(BASE_WIDTH/2 - 2*WHEEL_RADIUS)}"
@@ -60,5 +69,5 @@
   />
   <xacro:wheel
-    name_link="right_front_wheel" parent_link="base_link"
+    name_link="right_front_wheel" parent_link="chassis_link"
     mass="${WHEEL_MASS}" radius="${WHEEL_RADIUS}" width="${WHEEL_WIDTH}"
     translate_x="${BASE_WIDTH/2 - 2*WHEEL_RADIUS}"
@@ -67,5 +76,5 @@
   />
   <xacro:wheel
-    name_link="left_back_wheel" parent_link="base_link"
+    name_link="left_back_wheel" parent_link="chassis_link"
     mass="${WHEEL_MASS}" radius="${WHEEL_RADIUS}" width="${WHEEL_WIDTH}"
     translate_x="${-(BASE_WIDTH/2 - 2*WHEEL_RADIUS)}"
@@ -73,3 +82,8 @@
     translate_z="${-WHEEL_RADIUS}"
   />
+  <!-- Sensors -->
+  <xacro:hokuyo_laser
+    prefix="chassis" parent_link="chassis_link"
+    trans_x="0" trans_y="0" trans_z="${BASE_HEIGHT}"
+  />
 </robot>

Commit message: Add kinect_camera

File: simple4wd_description/urdf/simple4wd.urdf.xacro (robot description, xacro)
@@ -5,4 +5,5 @@
   <xacro:include filename="$(find simple4wd_description)/urdf/wheel.urdf.xacro" />
   <xacro:include filename="$(find simple4wd_description)/urdf/accessories/hokuyo_laser.urdf.xacro" />
+  <xacro:include filename="$(find simple4wd_description)/urdf/accessories/kinect_camera.urdf.xacro" />
   <!-- Gazebo Plugins -->
   <gazebo>
@@ -95,5 +96,8 @@
   <xacro:hokuyo_laser
     prefix="chassis" parent_link="chassis_link"
-    trans_x="0" trans_y="0" trans_z="${BASE_HEIGHT}"
+    trans_x="0" trans_y="0" trans_z="${BASE_HEIGHT * 2}"
   />
+  <xacro:kinect_camera prefix="kinect" parent_link="chassis_link">
+    <origin xyz="${BASE_LENGTH/2} 0 ${BASE_HEIGHT}" rpq="${PI} 0 0" />
+  </xacro:kinect_camera>
 </robot>
